File: KiCad/Capstone_Project_Mainboard/FPGA_Bank_0.kicad_sch (KiCad schematic)
At the start: 4 parts, among them U1 XC7K160T-FFG676_MIB

Commit message: Updated FPGA Footprint
Added die-to-pad length offsets to all pins of the FFG676 package. These values were derived from the delay files provided in Vivado.
+ Other minor bugfixes
Parts:
- U1: footprint Capstone_Library:Xilinx_FFG676_MOD -> Capstone_Library:Xilinx_FFG676_K7_160T
Changed lines of the file:
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@@
   (title_block
     (title "FPGA Bank 0 (Configuration) I/O")
-    (date "2023-12-18")
+    (date "2023-12-22")
     (rev "A")
     (company "Jordan Harris-Toovy")
@@
       (effects (font (size 1.27 1.27)) (justify right))
     )
-    (property "Footprint" "Capstone_Library:Xilinx_FFG676_MOD" (at 102.87 57.15 0)
-      (effects (font (size 1.27 1.27)) hide)
-    )
+    (property "Footprint" "Capstone_Library:Xilinx_FFG676_K7_160T" (at 102.87 57.15 0)
+      (effects (font (size 1.27 1.27)) hide)
+    )

Commit message: Core non-power parts defined
Most major non-power components added to KiCad project
Parts:
- R6: footprint (none) -> Resistor_SMD:R_0402_1005Metric; Part Number (none) -> RC0402FR-074K7L
- U1: Part Number (none) -> XC7K160T-2FFG676I
Connections:
- net FGPA_FLASH_SCK renamed FPGA_FLASH_SCK
Changed lines of the file:
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@@
   (title_block
     (title "FPGA Bank 0 (Configuration) I/O")
-    (date "2023-12-22")
+    (date "2023-12-26")
     (rev "A")
     (company "Jordan Harris-Toovy")
@@
     )
   )
-  (global_label "FGPA_FLASH_SCK" (shape bidirectional) (at 146.05 76.2 0) (fields_autoplaced)
+  (global_label "FPGA_FLASH_SCK" (shape bidirectional) (at 146.05 76.2 0) (fields_autoplaced)
     (effects (font (size 1 1) (color 65 65 65 1)) (justify left))
-    (property "Intersheetrefs" "${INTERSHEET_REFS}" (at 146.05 76.2 0)
-      (effects (font (size 1.27 1.27)) (justify right) hide)
+    (property "Intersheetrefs" "${INTERSHEET_REFS}" (at 161.9894 76.2 0)
+      (effects (font (size 1.27 1.27)) (justify left) hide)
     )
   )
@@
       (effects (font (size 1.27 1.27)) hide)
     )
-    (property "Datasheet" "" (at 102.87 60.96 0)
+    (property "Datasheet" "https://docs.xilinx.com/v/u/en-US/ds182_Kintex_7_Data_Sheet" (at 102.87 60.96 0)
+      (effects (font (size 1.27 1.27)) hide)
+    )
+    (property "Part Number" "XC7K160T-2FFG676I" (at 104.14 60.96 0)
       (effects (font (size 1.27 1.27)) hide)
     )
@@
       (effects (font (size 1.27 1.27)) (justify left))
     )
-    (property "Footprint" "" (at 201.676 76.454 90)
-      (effects (font (size 1.27 1.27)) hide)
-    )
-    (property "Datasheet" "~" (at 200.66 76.2 0)
+    (property "Footprint" "Resistor_SMD:R_0402_1005Metric" (at 201.676 76.454 90)
+      (effects (font (size 1.27 1.27)) hide)
+    )
+    (property "Datasheet" "https://www.mouser.com/datasheet/2/447/YAGEO_PYu_RC_Group_51_RoHS_L_12-3313492.pdf" (at 200.66 76.2 0)
+      (effects (font (size 1.27 1.27)) hide)
+    )
+    (property "Part Number" "RC0402FR-074K7L" (at 200.66 76.2 0)
       (effects (font (size 1.27 1.27)) hide)
     )
@@
       (effects (font (size 1.27 1.27)) (justify left))
     )
-    (property "Footprint" "" (at 191.516 76.454 90)
-      (effects (font (size 1.27 1.27)) hide)
-    )
-    (property "Datasheet" "~" (at 190.5 76.2 0)
+    (property "Footprint" "Resistor_SMD:R_0402_1005Metric" (at 191.516 76.454 90)
+      (effects (font (size 1.27 1.27)) hide)
+    )
+    (property "Datasheet" "https://www.mouser.com/datasheet/2/447/YAGEO_PYu_RC_Group_51_RoHS_L_12-3313492.pdf" (at 190.5 76.2 0)
+      (effects (font (size 1.27 1.27)) hide)
+    )
+    (property "Part Number" "RC0402FR-074K7L" (at 190.5 76.2 0)
       (effects (font (size 1.27 1.27)) hide)
     )
@@
       (effects (font (size 1.27 1.27)) (justify left))
     )
-    (property "Footprint" "" (at 181.356 76.454 90)
-      (effects (font (size 1.27 1.27)) hide)
-    )
-    (property "Datasheet" "~" (at 180.34 76.2 0)
-      (effects (font (size 1.27 1.27)) hide)
-    )
+    (property "Footprint" "Resistor_SMD:R_0402_1005Metric" (at 181.356 76.454 90)
+      (effects (font (size 1.27 1.27)) hide)
+    )
+    (property "Datasheet" "https://www.mouser.com/datasheet/2/447/YAGEO_PYu_RC_Group_51_RoHS_L_12-3313492.pdf" (at 180.34 76.2 0)
+      (effects (font (size 1.27 1.27)) hide)
+    )
+    (property "Part Number" "RC0402FR-074K7L" (at 180.34 76.2 0)
+      (effects (font (size 1.27 1.27)) hide)
+    )
