File: KiCad/Capstone_Project_Mainboard/FPGA_Banks_32_33_34.kicad_sch (KiCad schematic)
At the start: 1 part, among them U1 XC7K160T-FFG676_MIB

Commit message: Updated FPGA Footprint
Added die-to-pad length offsets to all pins of the FFG676 package. These values were derived from the delay files provided in Vivado.
+ Other minor bugfixes
Parts:
- U1: footprint Capstone_Library:Xilinx_FFG676_MOD -> Capstone_Library:Xilinx_FFG676_K7_160T
Changed lines of the file:
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@@
   (title_block
     (title "FPGA Banks 32 & 33 & 34 (HP) I/O")
-    (date "2023-12-18")
+    (date "2023-12-22")
     (rev "A")
     (company "Jordan Harris-Toovy")
@@
       (effects (font (size 1.27 1.27)) (justify right))
     )
-    (property "Footprint" "Capstone_Library:Xilinx_FFG676_MOD" (at 224.79 20.32 0)
+    (property "Footprint" "Capstone_Library:Xilinx_FFG676_K7_160T" (at 224.79 20.32 0)
       (effects (font (size 1.27 1.27)) hide)
     )
@@
       (effects (font (size 1.27 1.27)) (justify right))
     )
-    (property "Footprint" "Capstone_Library:Xilinx_FFG676_MOD" (at 52.07 20.32 0)
+    (property "Footprint" "Capstone_Library:Xilinx_FFG676_K7_160T" (at 52.07 20.32 0)
       (effects (font (size 1.27 1.27)) hide)
     )
@@
       (effects (font (size 1.27 1.27)) (justify right))
     )
-    (property "Footprint" "Capstone_Library:Xilinx_FFG676_MOD" (at 138.43 20.32 0)
-      (effects (font (size 1.27 1.27)) hide)
-    )
+    (property "Footprint" "Capstone_Library:Xilinx_FFG676_K7_160T" (at 138.43 20.32 0)
+      (effects (font (size 1.27 1.27)) hide)
+    )

Commit message: Core non-power parts defined
Most major non-power components added to KiCad project
Parts:
- U1: Part Number (none) -> XC7K160T-2FFG676I
Changed lines of the file:
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@@
   (title_block
     (title "FPGA Banks 32 & 33 & 34 (HP) I/O")
-    (date "2023-12-22")
+    (date "2023-12-26")
     (rev "A")
     (company "Jordan Harris-Toovy")
@@
       (effects (font (size 1.27 1.27)) hide)
     )
-    (property "Datasheet" "" (at 224.79 24.13 0)
+    (property "Datasheet" "https://docs.xilinx.com/v/u/en-US/ds182_Kintex_7_Data_Sheet" (at 224.79 24.13 0)
+      (effects (font (size 1.27 1.27)) hide)
+    )
+    (property "Part Number" "XC7K160T-2FFG676I" (at 226.06 24.13 0)
       (effects (font (size 1.27 1.27)) hide)
     )
@@
       (effects (font (size 1.27 1.27)) hide)
     )
-    (property "Datasheet" "" (at 52.07 24.13 0)
+    (property "Datasheet" "https://docs.xilinx.com/v/u/en-US/ds182_Kintex_7_Data_Sheet" (at 52.07 24.13 0)
+      (effects (font (size 1.27 1.27)) hide)
+    )
+    (property "Part Number" "XC7K160T-2FFG676I" (at 53.34 24.13 0)
       (effects (font (size 1.27 1.27)) hide)
     )
@@
       (effects (font (size 1.27 1.27)) hide)
     )
-    (property "Datasheet" "" (at 138.43 24.13 0)
-      (effects (font (size 1.27 1.27)) hide)
-    )
+    (property "Datasheet" "https://docs.xilinx.com/v/u/en-US/ds182_Kintex_7_Data_Sheet" (at 138.43 24.13 0)
+      (effects (font (size 1.27 1.27)) hide)
+    )
+    (property "Part Number" "XC7K160T-2FFG676I" (at 139.7 24.13 0)
+      (effects (font (size 1.27 1.27)) hide)
+    )
